File: projects/UWRT/powerSupply/power_supply.brd (EAGLE design)
At the start: 101.6 x 101.6 mm, 68 parts, among them IC1 NE555, U1 SN74HC595PW

Commit message: Updated semi - final design
Parts:
- removed IC1: NE555, st-microelectronics:DIL-08
- removed VBATIN_R2, VBATIN_R3, VBATIN_R4: 330, SparkFun-Resistors:0603
- added 555TIMER: NE555, st-microelectronics:DIL-08
- added CANH_OUT_R, CANL_OUT_R: 60, SparkFun-Resistors:0603
- added CAN_SPLIT_C: 4700pF, capacitor-wima:C2.5-2
- added OSC1_C: 1nF, capacitor-wima:C2.5-2
- added OSC2_C: 1 nF, capacitor-wima:C2.5-2
- added Q1: (no value), crystal:HC49/S
- moved C_555_2 104.1 mm to (73.0, 29.4), turned to 180 degrees
- moved C_555_1 96.0 mm to (84.1, 21.4), turned to 270 degrees
- moved R_555_VCC 79.6 mm to (70.6, 21.4), turned to 90 degrees
- moved MCP2561 2.38 mm to (81.0, 39.7)
- moved C9_3V 0.79 mm to (60.3, 51.6)
Connections:
- removed net N$2: IC1.2, R_555_VCC.1
- removed net N$3: C_555_1.1, IC1.5
- removed net N$6: C_555_2.1, IC1.6, IC1.7
- removed net N$7: IC1.4, IC1.8, R_555_VCC.2
- new net 555_CON: 555TIMER.5, C_555_1.1
- new net 555_TREDIS: 555TIMER.6, 555TIMER.7, C_555_2.1
- new net 555_TRIG: 555TIMER.2, R_555_VCC.1
- new net CAN_SPLIT: CANH_OUT_R.2, CANL_OUT_R.1, CAN_SPLIT_C.1, MCP2561.P$5
- new net OSC1: OSC1_C.2, Q1.2, U$2.8
- new net OSC2: OSC2_C.2, Q1.1, U$2.9
- net CANH_OUT: now also CANH_OUT_R.1
- net CANL_OUT: now also CANL_OUT_R.2
- net GND: now also 555TIMER.1, CAN_SPLIT_C.2, C_555_2.2, OSC1_C.1, OSC2_C.1; no longer IC1.1
- net OUT555: now also 555TIMER.3; no longer IC1.3
- net VCC: now also 555TIMER.4, 555TIMER.8, R_555_VCC.2
Routing:
- net VCC: track 261.5 -> 169.9 mm, vias 6 -> 5
- net OSC2: track 0.00 -> 14.8 mm
- net CAN_SPLIT: track 0.00 -> 13.1 mm
- net OSC1: track 0.00 -> 9.17 mm
- net 555_TREDIS: track 0.00 -> 7.26 mm
- net 555_TRIG: track 0.00 -> 6.31 mm
- net CANH_OUT: track 144.6 -> 149.9 mm
- net 555_CON: track 0.00 -> 4.39 mm
- net CANL_OUT: track 139.1 -> 141.7 mm
- net OUT555: track 15.0 -> 12.9 mm
- net N$8: track 3.48 -> 4.80 mm
- net N$14: track 2.94 -> 3.83 mm

Commit message: Error checking, version 1.0 to print
Routing:
- net VCC: track 169.9 -> 206.8 mm
Changed lines of the file:
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@@
 <wire x1="53.18125" y1="93.6625" x2="56.35625" y2="93.6625" width="0.1524" layer="1"/>
 <wire x1="56.35625" y1="93.6625" x2="61.11875" y2="98.425" width="0.1524" layer="1"/>
-<wire x1="44.36" y1="33.02" x2="43.97375" y2="33.02" width="0.508" layer="1"/>
+<wire x1="43.97375" y1="33.02" x2="44.36" y2="33.02" width="0.508" layer="1"/>
 <wire x1="43.97375" y1="33.02" x2="39.6875" y2="37.30625" width="0.508" layer="1"/>
 <wire x1="39.6875" y1="37.30625" x2="34.13125" y2="37.30625" width="0.508" layer="1"/>
@@
 <wire x1="13.3985" y1="21.9075" x2="38.57625" y2="21.9075" width="0.508" layer="1"/>
 <wire x1="38.57625" y1="21.9075" x2="38.89375" y2="22.225" width="0.508" layer="1"/>
+<wire x1="44.36" y1="33.02" x2="44.36" y2="19.49544375" width="0.508" layer="1"/>
+<wire x1="44.36" y1="19.49544375" x2="43.147" y2="18.28244375" width="0.508" layer="1"/>
+<wire x1="43.147" y1="8.222" x2="42.8625" y2="7.9375" width="0.508" layer="1"/>
+<wire x1="43.147" y1="18.28244375" x2="43.147" y2="8.222" width="1.016" layer="1"/>
+<wire x1="54.8005" y1="3.175" x2="53.975" y2="7.9375" width="0.508" layer="1"/>
+<wire x1="53.975" y1="7.9375" x2="52.3875" y2="7.9375" width="0.508" layer="1"/>
+<wire x1="52.3875" y1="7.9375" x2="52.2605" y2="3.175" width="0.508" layer="1"/>
 <wire x1="39.6875" y1="37.30625" x2="40.9575" y2="45.025" width="0" layer="19" extent="1-16"/>
-<wire x1="54.8005" y1="3.175" x2="55.5625" y2="20.0025" width="0" layer="19" extent="1-1"/>
-<wire x1="52.2605" y1="3.175" x2="54.8005" y2="3.175" width="0" layer="19" extent="1-1"/>
 </signal>
 <signal name="V_BAT_BAL+">
@@
 <wire x1="84.7925" y1="34.5775" x2="84.7925" y2="37.445" width="0.1524" layer="1"/>
 <wire x1="84.7925" y1="37.445" x2="84.1375" y2="38.1" width="0.1524" layer="1"/>
-<wire x1="77.875" y1="96.8375" x2="77.875" y2="100.0125" width="0" layer="19" extent="1-1"/>
-<wire x1="60.325" y1="92.075" x2="76.2" y2="96.8375" width="0" layer="19" extent="1-1"/>
-<wire x1="46.0375" y1="92.075" x2="58.65" y2="92.075" width="0" layer="19" extent="1-1"/>
-<wire x1="37.30625" y1="96.8375" x2="44.3625" y2="92.075" width="0" layer="19" extent="1-1"/>
-<wire x1="59.53125" y1="75.72375" x2="58.65" y2="92.075" width="0" layer="19" extent="1-1"/>
-<wire x1="63.1825" y1="75.625" x2="59.53125" y2="75.72375" width="0" layer="19" extent="16-16"/>
-<wire x1="53.18125" y1="76.5175" x2="59.53125" y2="75.72375" width="0" layer="19" extent="1-1"/>
-<wire x1="49.2125" y1="75.565" x2="53.18125" y2="76.5175" width="0" layer="19" extent="1-1"/>
-<wire x1="44.45" y1="74.295" x2="49.2125" y2="75.565" width="0" layer="19" extent="1-1"/>
-<wire x1="42.8625" y1="61.2775" x2="44.45" y2="74.295" width="0" layer="19" extent="1-1"/>
-<wire x1="39.28" y1="56.8325" x2="42.8625" y2="61.2775" width="0" layer="19" extent="1-1"/>
-<wire x1="43.4975" y1="50.225" x2="39.28" y2="56.8325" width="0" layer="19" extent="16-16"/>
-<wire x1="44.7675" y1="50.225" x2="43.4975" y2="50.225" width="0" layer="19" extent="16-16"/>
-<wire x1="44.7675" y1="45.025" x2="44.7675" y2="50.225" width="0" layer="19" extent="16-16"/>
-<wire x1="50.8" y1="47.3075" x2="44.7675" y2="45.025" width="0" layer="19" extent="16-16"/>
-<wire x1="57.15" y1="45.4025" x2="50.8" y2="47.3075" width="0" layer="19" extent="1-1"/>
-<wire x1="60.325" y1="50.32375" x2="57.15" y2="45.4025" width="0" layer="19" extent="1-1"/>
-<wire x1="43.4975" y1="36.5125" x2="44.7675" y2="45.025" width="0" layer="19" extent="16-16"/>
-<wire x1="39.28" y1="33.02" x2="43.4975" y2="36.5125" width="0" layer="19" extent="1-1"/>
-<wire x1="40.9575" y1="22.8" x2="39.28" y2="23.405" width="0" layer="19" extent="16-16"/>
-<wire x1="42.2275" y1="22.8" x2="40.9575" y2="22.8" width="0" layer="19" extent="16-16"/>
-<wire x1="40.9575" y1="28" x2="39.28" y2="23.405" width="0" layer="19" extent="16-16"/>
-<wire x1="53.975" y1="36.83" x2="57.15" y2="45.4025" width="0" layer="19" extent="1-1"/>
-<wire x1="55.245" y1="30.1625" x2="53.975" y2="36.83" width="0" layer="19" extent="1-1"/>
-<wire x1="61.595" y1="30.1625" x2="55.245" y2="30.1625" width="0" layer="19" extent="1-1"/>
-<wire x1="60.325" y1="34.29" x2="61.595" y2="30.1625" width="0" layer="19" extent="1-1"/>
-<wire x1="64.29375" y1="36.03625" x2="60.325" y2="34.29" width="0" layer="19" extent="1-1"/>
-<wire x1="65.405" y1="32.54375" x2="64.29375" y2="36.03625" width="0" layer="19" extent="1-1"/>
-<wire x1="71.755" y1="34.13125" x2="65.405" y2="32.54375" width="0" layer="19" extent="1-1"/>
-<wire x1="71.755" y1="29.36875" x2="71.755" y2="34.13125" width="0" layer="19" extent="1-1"/>
-<wire x1="63.5" y1="22.5425" x2="61.595" y2="30.1625" width="0" layer="19" extent="1-1"/>
-<wire x1="58.7375" y1="20.0025" x2="63.5" y2="22.5425" width="0" layer="19" extent="1-1"/>
-<wire x1="69.85" y1="50.4825" x2="60.325" y2="50.32375" width="0" layer="19" extent="1-1"/>
-<wire x1="52.86375" y1="57.15" x2="50.8" y2="47.3075" width="0" layer="19" extent="1-1"/>
-<wire x1="73.18375" y1="17.62125" x2="63.5" y2="22.5425" width="0" layer="19" extent="1-1"/>
-<wire x1="84.1375" y1="20.16125" x2="73.18375" y2="17.62125" width="0" layer="19" extent="1-1"/>
-<wire x1="87.4395" y1="20.0025" x2="84.1375" y2="20.16125" width="0" layer="19" extent="1-1"/>
-<wire x1="83.185" y1="27.178" x2="84.1375" y2="20.16125" width="0" layer="19" extent="16-16"/>
-<wire x1="84.7925" y1="34.5775" x2="83.185" y2="27.178" width="0" layer="19" extent="1-16"/>
 </signal>
 <signal name="N$14">
@@
 <contactref element="MCP2561" pad="P$6"/>
 <contactref element="CANL_OUT_R" pad="2"/>
-<wire x1="79.18245" y1="33.686025" x2="79.18245" y2="33.687075" width="0" layer="19" extent="1-16"/>
 <wire x1="81.75625" y1="11.1125" x2="81.75625" y2="12.7" width="0.1524" layer="1"/>
 <wire x1="81.75625" y1="11.1125" x2="80.9625" y2="10.31875" width="0.1524" layer="1"/>
@@
 <wire x1="81.358725" y1="33.3375" x2="81.75625" y2="33.735025" width="0.1524" layer="1"/>
 <wire x1="85.725" y1="96.8375" x2="84.9875" y2="96.8375" width="0" layer="19" extent="1-16"/>
-<wire x1="79.18245" y1="33.686025" x2="78.6375" y2="33.3375" width="0" layer="19" extent="1-1"/>
 </signal>
 <signal name="N$16">

Commit message: Updated to add the gerbers
Parts:
- moved CANH_LED 3.37 mm to (81.8, 97.6)
- moved CANH_R 3.37 mm to (86.5, 97.6)
- moved CANL_LED 2.86 mm to (81.8, 95.2)
- moved CANL_R 2.86 mm to (86.5, 95.2)
- flipped R7 to the top
- renumbered U$5 to POWER_IN
Routing:
- net 3.3V_OUT: track 162.1 -> 168.0 mm
- net GND: track 156.3 -> 161.1 mm
- net CANH_OUT: track 149.9 -> 145.9 mm, vias 1 -> 2
- net CANL_OUT: track 141.7 -> 138.0 mm, vias 1 -> 2
- net 12V_GND: track 180.3 -> 183.2 mm
- net 12V_CON_ONOFF: track 170.3 -> 173.0 mm, vias 4 -> 6
- net VCC: track 206.8 -> 209.0 mm, vias 5 -> 6
- net N$8: track 4.80 -> 3.16 mm
Other:
- board text added: "12V Current"
- board text added: "12V Out"
- board text added: "12V Voltage"
- board text added: "3.3V Current"
- board text added: "3.3V Out"
- board text added: "3.3V Voltage"
- board text added: "CAN High"
- board text added: "CAN Low"
- board text added: "Power In"
- board text added: "Underwater Robotics At The Ohio State University Power Converter Board"
- board text added: "VCC Current"
- board text added: "VCC Out"
- board text added: "VCC Voltage"
