File: projects/UWRT/powerSupply/power_supply.sch (EAGLE design)
At the start: 68 parts, among them IC1 NE555, U1 SN74HC595PW

Commit message: Updated semi - final design
Parts:
- removed VBATIN_R2, VBATIN_R3, VBATIN_R4: 330, SparkFun-Resistors:0OHM-0603-1/10W-5%
- added CANH_OUT_R, CANL_OUT_R: 60, SparkFun-Resistors:0OHM-0603-1/10W-5%
- added CAN_SPLIT_C: 4700pF, capacitor-wima:C2.5/2
- added OSC1_C: 1nF, capacitor-wima:C2.5/2
- added OSC2_C: 1 nF, capacitor-wima:C2.5/2
- added Q1: (no value), crystal:CRYSTALHC49S
- renumbered IC1 to 555TIMER
Connections:
- net N$2 renamed 555_TRIG
- net N$3 renamed 555_CON
- net N$6 renamed 555_TREDIS
- removed net N$7: 555TIMER./RES, 555TIMER.VCC+, R_555_VCC.2
- new net CAN_SPLIT: CANH_OUT_R.2, CANL_OUT_R.1, CAN_SPLIT_C.1, MCP2561.SPLIT
- new net OSC1: OSC1_C.2, Q1.2, U$2.OSC1/CLKIN
- new net OSC2: OSC2_C.2, Q1.1, U$2.OSC2
- net CANH_OUT: now also CANH_OUT_R.1
- net CANL_OUT: now also CANL_OUT_R.2
- net GND: now also CAN_SPLIT_C.2, C_555_2.2, OSC1_C.1, OSC2_C.1
- net VCC: now also 555TIMER./RES, 555TIMER.VCC+, R_555_VCC.2
Other:
- moved on the sheet: C_555_2

Commit message: Updated to add the gerbers
Parts:
- renumbered U$5 to POWER_IN
Changed lines of the file:
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@@
 <part name="SUPPLY15" library="supply2" library_urn="urn:adsk.eagle:library:372" deviceset="GND" device=""/>
 <part name="P+8" library="supply1" library_urn="urn:adsk.eagle:library:371" deviceset="VCC" device=""/>
-<part name="GND1" library="supply1" library_urn="urn:adsk.eagle:library:371" deviceset="GND" device=""/>
+<part name="V_BAT_BAL-" library="supply1" library_urn="urn:adsk.eagle:library:371" deviceset="GND" device=""/>
 <part name="12V_OUT_TP" library="testpad" library_urn="urn:adsk.eagle:library:385" deviceset="PTR1" device="B1,27"/>
 <part name="TP2" library="testpad" library_urn="urn:adsk.eagle:library:385" deviceset="PTR1" device="B1,27"/>
@@
 <part name="P+9" library="supply1" library_urn="urn:adsk.eagle:library:371" deviceset="VCC" device=""/>
 <part name="P+10" library="supply1" library_urn="urn:adsk.eagle:library:371" deviceset="VCC" device=""/>
-<part name="U$5" library="molex" deviceset="39-30-1020" device=""/>
+<part name="POWER_IN" library="molex" deviceset="39-30-1020" device=""/>
 <part name="U$6" library="molex" deviceset="39-30-1040" device=""/>
 <part name="U$7" library="molex" deviceset="70555-0003" device=""/>
@@
 <instance part="SUPPLY15" gate="GND" x="662.94" y="187.96"/>
 <instance part="P+8" gate="VCC" x="685.8" y="238.76"/>
-<instance part="GND1" gate="1" x="320.04" y="162.56"/>
+<instance part="V_BAT_BAL-" gate="1" x="320.04" y="162.56"/>
 <instance part="12V_OUT_TP" gate="G$1" x="459.74" y="289.56" rot="R180"/>
 <instance part="TP2" gate="G$1" x="464.82" y="236.22" rot="R180"/>
@@
 <instance part="P+9" gate="VCC" x="581.66" y="185.42"/>
 <instance part="P+10" gate="VCC" x="622.3" y="185.42"/>
-<instance part="U$5" gate="G$1" x="297.18" y="223.52" rot="R90"/>
+<instance part="POWER_IN" gate="G$1" x="297.18" y="223.52" rot="R90"/>
 <instance part="U$6" gate="G$1" x="487.68" y="314.96" rot="MR0"/>
 <instance part="U$7" gate="G$1" x="447.04" y="116.84"/>
@@
 <pinref part="5V_CONVERTER" gate="G$1" pin="+VIN"/>
 <wire x1="322.58" y1="223.52" x2="391.16" y2="223.52" width="0.1524" layer="91"/>
-<pinref part="3.3V_CONVERTER" gate="G$1" pin="+VIN"/>
-<wire x1="391.16" y1="170.18" x2="322.58" y2="170.18" width="0.1524" layer="91"/>
 <wire x1="322.58" y1="170.18" x2="322.58" y2="223.52" width="0.1524" layer="91"/>
 <junction x="322.58" y="223.52"/>
@@
 <wire x1="353.06" y1="284.48" x2="322.58" y2="284.48" width="0.1524" layer="91"/>
 <wire x1="322.58" y1="284.48" x2="322.58" y2="228.6" width="0.1524" layer="91"/>
-<pinref part="U$5" gate="G$1" pin="2"/>
+<pinref part="POWER_IN" gate="G$1" pin="2"/>
 <wire x1="322.58" y1="228.6" x2="322.58" y2="223.52" width="0.1524" layer="91"/>
 <junction x="322.58" y="228.6"/>
@@
 <wire x1="309.88" y1="236.22" x2="289.56" y2="236.22" width="0.1524" layer="91"/>
 <wire x1="289.56" y1="236.22" x2="289.56" y2="228.6" width="0.1524" layer="91"/>
+<pinref part="3.3V_CONVERTER" gate="G$1" pin="+VIN"/>
+<wire x1="322.58" y1="170.18" x2="391.16" y2="170.18" width="0.1524" layer="91"/>
 </segment>
 </net>
@@
 <wire x1="353.06" y1="264.16" x2="320.04" y2="264.16" width="0.1524" layer="91"/>
 <wire x1="320.04" y1="264.16" x2="320.04" y2="220.98" width="0.1524" layer="91"/>
-<pinref part="GND1" gate="1" pin="GND"/>
+<pinref part="V_BAT_BAL-" gate="1" pin="GND"/>
 <wire x1="320.04" y1="165.1" x2="320.04" y2="167.64" width="0.1524" layer="91"/>
 <junction x="320.04" y="167.64"/>
-<pinref part="U$5" gate="G$1" pin="1"/>
+<pinref part="POWER_IN" gate="G$1" pin="1"/>
 <wire x1="297.18" y1="218.44" x2="309.88" y2="218.44" width="0.1524" layer="91"/>
 <junction x="320.04" y="218.44"/>
