File: projects/uwrt/coProcessor/pinconnections.sch (EAGLE design)
At the start: 26 parts, among them U1 MPU-9250, U3 HTU21D

Commit message: Merged template with coPro connections
Parts:
- removed CANH_LED, CANL_LED: (no value), SparkFun-LED:LED1206
- removed CANH_OUT_R, CANL_OUT_R: 60, SparkFun-Resistors:0OHM-0603-1/10W-5%
- removed CANH_R, CANL_R: 330, SparkFun-Resistors:0OHM-0603-1/10W-5%
- removed CAN_SPLIT_C: 4700pF, capacitor-wima:C2.5/2
- removed MCP2561: MCP2561, MCP2561:MCP2561
- removed U$7: 70555-0003, molex:70555-0003
- added U2: MCP2551, SparkFun-IC-Comms:MCP2551
- U$4: value 5530843-6-STS -> MCP2561; device te-connectivity:5530843-6-STS -> MCP2561:MCP2561
Connections:
- removed net +5V: MCP2561.VDD, U$4.5V, U$7.3
- removed net 12V_OUT: U$4.12V+, U$7.4
- removed net CANH_LED: CANH_LED.A, CANH_R.1
- removed net CANH_OUT: CANH_OUT_R.1, CANH_R.2, MCP2561.CANH, U$4.CAN_H
- removed net CANL_LED: CANL_LED.A, CANL_R.2
- removed net CANL_OUT: CANL_OUT_R.2, CANL_R.1, MCP2561.CANL, U$4.CAN_L
- removed net CAN_RX: MCP2561.RXD, U$1.44
- removed net CAN_SPLIT: CANH_OUT_R.2, CANL_OUT_R.1, CAN_SPLIT_C.1, MCP2561.SPLIT
- removed net CAN_TX: MCP2561.TXD, U$1.45
- removed net N$15: U$4.12V-
- removed net N$2 (its old number): R2.1, U$1.59
- new net N$5: U$1.44, U2.RXD
- new net N$6: U2.CANL
- new net N$7: U2.CANH
- new net SCL: R1.1, U$1.58, U$2.SCL/SPC, U$3.SCL, U1.SCL/SCLK, U3.SCK
- new net SDA: R2.1, U$1.59, U$2.SDA/SDI, U$3.SDA, U1.SDA/SDI, U3.DATA
- new net VDD: C2.1, C3.1, C4.1, C5.1, C6.1, C9.1, R1.2, R2.2, U$1.13, U$1.19, U$1.64, U$2.CS, U$2.SA0/SDO, U$2.VDD, U$2.VDD_IO, U$3.VCC, U1.!CS, U1.AD0/SDO, U1.VDD, U1.VDDIO, U2.VDD, U3.VDD
- net +3V3: no longer C2.1, C3.1, C4.1, C5.1, C6.1, C9.1, R1.2, R2.2, U$1.13, U$1.19, U$1.64, U$2.VDD, U$2.VDD_IO, U$4.3V3, U$7.2, U1.VDD, U1.VDDIO, U3.VDD
- net GND: now also U$3.WP, U2.VSS; no longer CANH_LED.C, CANL_LED.C, CAN_SPLIT_C.2, MCP2561.STBY, MCP2561.VSS, U$4.GND, U$7.1
- net N$3: now also U$1.45, U2.TXD; no longer R1.1, U$1.58
Other:
- moved on the sheet: C1, C2, C3, C4, C5, C6, C7, C8, C9, R1, R2, U$1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
