File: projects/uwrt/coProcessor/co_processor.sch (EAGLE design)
At the start: 26 parts, among them U1 MPU-9250, U3 HTU21D

Commit message: Added coPro decoupling power stuff
Parts:
- added C10, C11, C12, C13, C14: 100nF, rcl:C-EU025-025X050
- added C15: 1uF, rcl:C-EU025-025X050
- added DEPTH_SENSOR: DF13-4P-1.25DSA, con-hirose-df13:DF13-4P-1.25DSA
- added JTAG_HEADER: M05X2-50MIL_SHROUD, Connectors:M05X2-50MIL_SHROUD
- added PWM, PWM1, PWM2, PWM3, PWM4, PWM5, PWM6, PWM7, PWM8, PWM9: (no value), con-lstb:MA03-1
- added PWM_LED, PWM_LED1, PWM_LED2, PWM_LED3, PWM_LED4, PWM_LED5, PWM_LED6, PWM_LED7, PWM_LED8, PWM_LED9: (no value), SparkFun-LED:LED1206
- added PWM_R, PWM_R1, PWM_R2, PWM_R3, PWM_R4, PWM_R5, PWM_R6, PWM_R7, PWM_R8, PWM_R9: 330, SparkFun-Resistors:0OHM-0603-1/10W-5%
- renumbered U$1 to STM32F405
Connections:
- net N$10 renamed VCAP_1
- net N$11 renamed VCAP_2
- removed net N$3: R1.1, STM32F405.58
- new net GND1: JTAG_HEADER.3, JTAG_HEADER.5, JTAG_HEADER.9
- new net I2C_SCL: DEPTH_SENSOR.2, R2.1, STM32F405.61
- new net I2C_SDA: DEPTH_SENSOR.3, R1.1, STM32F405.62
- new net N$13: PWM_LED2.A, PWM_R2.2
- new net N$14: PWM_LED3.A, PWM_R3.2
- new net N$17: PWM_LED4.A, PWM_R4.2
- new net N$18: PWM_LED5.A, PWM_R5.2
- new net N$19: PWM_LED6.A, PWM_R6.2
- new net N$20: PWM_LED7.A, PWM_R7.2
- new net N$21: PWM_LED8.A, PWM_R8.2
- new net N$22: PWM_LED9.A, PWM_R9.2
- new net N$7: PWM_LED.A, PWM_R.2
- new net N$8: PWM_LED1.A, PWM_R1.2
- new net PWM0_OUT: PWM.3, PWM_R.1, STM32F405.30
- new net PWM1_OUT: PWM1.3, PWM_R1.1, STM32F405.29
- new net PWM2_OUT: PWM2.3, PWM_R2.1, STM32F405.27
- new net PWM3_OUT: PWM3.3, PWM_R3.1, STM32F405.26
- new net PWM4_OUT: PWM4.3, PWM_R4.1, STM32F405.23
- new net PWM5_OUT: PWM5.3, PWM_R5.1, STM32F405.22
- new net PWM6_OUT: PWM6.3, PWM_R6.1, STM32F405.17
- new net PWM7_OUT: PWM7.3, PWM_R7.1, STM32F405.16
- new net PWM8_OUT: PWM8.3, PWM_R8.1, STM32F405.15
- new net PWM9_OUT: PWM9.3, PWM_R9.1, STM32F405.14
- new net TCK: JTAG_HEADER.4
- new net TMS: JTAG_HEADER.2
- new net VCC: JTAG_HEADER.1
- net +3V3: now also C10.1, C12.1, C13.1, C14.1, C15.1, DEPTH_SENSOR.1
- net GND: now also C10.2, C11.1, C11.2, C12.2, C13.2, C14.2, C15.2, DEPTH_SENSOR.4, PWM_LED.C, PWM_LED1.C, PWM_LED2.C, PWM_LED3.C, PWM_LED4.C, PWM_LED5.C, PWM_LED6.C, PWM_LED7.C, PWM_LED8.C, PWM_LED9.C
- net N$2: now also JTAG_HEADER.10; no longer R2.1, STM32F405.59
Other:
- note added: "PWM output goes to Pin 3, GND to pin 1"
- moved on the sheet: C1, C2, C3, C4, C5, C6, C7, C8, CANH_LED, CANH_OUT_R, CANH_R, CANL_LED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

Commit message: No frills processing board revision 1.0.0
Parts:
- removed C1, C2: 0.1uF, rcl:C-EU025-025X050
- removed C3: 10nF, rcl:C-EU025-025X050
- removed C4: 100uF, rcl:C-EU025-025X050
- removed C5: 4.7uF, rcl:C-EU025-025X050
- removed C6: 100nF, rcl:C-EU025-025X050
- removed JTAG_HEADER: M05X2-50MIL_SHROUD, Connectors:M05X2-50MIL_SHROUD
- removed U$2: LPS25H, st-microelectronics:LPS25H
- removed U$3: 24AA02, microchip:24AA02
- removed U1: MPU-9250, SparkFun-Sensors:MPU-9250
- removed U3: HTU21D, SparkFun-Sensors:HTU21D
- added HB_R, HB_R1: 330, SparkFun-Resistors:0OHM-0603-1/10W-5%
- added JTAG: (no value), pinhead:PINHD-2X10
- added MICROSD: MICRO-SD_CARD_SOCKET, SparkFun-Connectors:MICRO-SD_CARD_SOCKET
- added MINI_USB_B: USB_MINI-B_SMT, SparkFun-Connectors:USB_MINI-B_SMT
- added OSC1_C: 1nF, capacitor-wima:C2.5/2
- added OSC2_C: 1 nF, capacitor-wima:C2.5/2
- added Q1: (no value), crystal:CRYSTALHC49S
- added RESET_SWITCH: (no value), switch-omron:10-XX
- added STATUS_1, STATUS_2: (no value), SparkFun-LED:LED1206
- added SWITCHES: 39-30-1040, molex:39-30-1040
Connections:
- removed net GND1: JTAG_HEADER.3, JTAG_HEADER.5, JTAG_HEADER.9
- removed net N$6: U1.GND
- removed net N$9: C1.1, U1.REGOUT
- removed net TCK: JTAG_HEADER.4
- removed net TMS: JTAG_HEADER.2
- removed net VCC: JTAG_HEADER.1
- new net GND_ESC: PWM.1, PWM1.1, PWM2.1, PWM3.1, PWM4.1, PWM5.1, PWM6.1, PWM7.1, PWM8.1, PWM9.1, PWM_LED.C, PWM_LED1.C, PWM_LED2.C, PWM_LED3.C, PWM_LED4.C, PWM_LED5.C, PWM_LED6.C, PWM_LED7.C, PWM_LED8.C, PWM_LED9.C
- new net HB_OUT: HB_R.1, STM32F405.38
- new net HB_OUT1: HB_R1.1, STM32F405.37
- new net JTAG_RST: JTAG.3, STM32F405.56
- new net JTAG_TCK: JTAG.9, STM32F405.49
- new net JTAG_TDI: JTAG.5, STM32F405.50
- new net JTAG_TDO: JTAG.13, STM32F405.55
- new net JTAG_TMS: JTAG.7, STM32F405.46
- new net KILL_SW: STM32F405.34, SWITCHES.2
- new net N$3: HB_R1.2, STATUS_2.A
- new net NRST: JTAG.15, RESET_SWITCH.P, RESET_SWITCH.P1, STM32F405.7
- new net OSC_IN: OSC1_C.2, Q1.1, STM32F405.5
- new net OSC_OUT: OSC2_C.2, Q1.2, STM32F405.6
- new net SDIO_CK: MICROSD.SCK, STM32F405.53
- new net SDIO_CMD: MICROSD.!CS, STM32F405.54
- new net SDIO_D0: MICROSD.DO, STM32F405.39
- new net START_SW: STM32F405.33, SWITCHES.1
- new net USB_DM: MINI_USB_B.D-, STM32F405.36
- new net USB_DP: MINI_USB_B.D+, STM32F405.35
- net +3V3: now also C11.1, JTAG.1, JTAG.2, MICROSD.VCC, MINI_USB_B.VBUS, SWITCHES.3, SWITCHES.4; no longer C2.1, C3.1, C4.1, C5.1, C6.1, U$2.VDD, U$2.VDD_IO, U1.VDD, U1.VDDIO, U3.VDD
- net GND: now also JTAG.10, JTAG.12, JTAG.14, JTAG.16, JTAG.18, JTAG.20, JTAG.4, JTAG.6, JTAG.8, MICROSD.CD1, MICROSD.CD2, MICROSD.GND, MICROSD.SHIELD@1, MICROSD.SHIELD@3, MINI_USB_B.GND, MINI_USB_B.SHIELD, OSC1_C.1, OSC2_C.1, RESET_SWITCH.S1, STATUS_1.C, STATUS_2.C; no longer C1.2, C11.1, C2.2, C3.2, C4.2, C5.2, C6.2, PWM_LED.C, PWM_LED1.C, PWM_LED2.C, PWM_LED3.C, PWM_LED4.C, PWM_LED5.C, PWM_LED6.C, PWM_LED7.C, PWM_LED8.C, PWM_LED9.C, U$2.GND1, U$2.GND2, U$2.RES, U$3.VSS, U3.GND@2, U3.GND@7
- net N$2: now also HB_R.2, STATUS_1.A; no longer JTAG_HEADER.10
Other:
- moved on the sheet: CANH_LED, CANH_OUT_R, CANH_R, CANL_LED, CANL_OUT_R, CANL_R, CAN_SPLIT_C

Commit message: No frills Co Processing board rev 1.1.0
Parts:
- removed PWM, PWM1, PWM2, PWM3, PWM4, PWM5, PWM6, PWM7, PWM8, PWM9: (no value), con-lstb:MA03-1
- added BIAS_R, BIAS_R1, BIAS_R2, BIAS_R3, BIAS_R4, BIAS_R5, BIAS_R6, BIAS_R7, BIAS_R8, BIAS_R9: 1K, SparkFun-Resistors:0OHM-0603-1/10W-5%
- added OPI_PWM0, OPI_PWM1, OPI_PWM2, OPI_PWM3, OPI_PWM4, OPI_PWM5, OPI_PWM6, OPI_PWM7, OPI_PWM8, OPI_PWM9: SFH610, SFH610:SFH610
- added P0, P1, P2, P3, P4, P5, P6, P7, P8, P9: (no value), con-lstb:MA03-1
- added PWM_IN0, PWM_IN1, PWM_IN2, PWM_IN3, PWM_IN4, PWM_IN5, PWM_IN6, PWM_IN7, PWM_IN8, PWM_IN9: 330, SparkFun-Resistors:0OHM-0603-1/10W-5%
Connections:
- new net N$10: OPI_PWM4.A, PWM_IN4.2
- new net N$11: OPI_PWM5.A, PWM_IN5.2
- new net N$17: OPI_PWM9.A, PWM_IN9.2
- new net N$23: OPI_PWM6.A, PWM_IN6.2
- new net N$24: OPI_PWM7.A, PWM_IN7.2
- new net N$25: OPI_PWM8.A, PWM_IN8.2
- new net N$29: OPI_PWM0.A, PWM_IN0.2
- new net N$47: OPI_PWM2.A, PWM_IN2.2
- new net N$6: OPI_PWM1.A, PWM_IN1.2
- new net N$9: OPI_PWM3.A, PWM_IN3.2
- new net PWM0_BO: BIAS_R.1, OPI_PWM0.COL, P0.3, PWM_R.1
- new net PWM1_BO: BIAS_R1.1, OPI_PWM1.COL, P1.3, PWM_R1.1
- new net PWM2_BO: BIAS_R2.1, OPI_PWM2.COL, P2.3, PWM_R2.1
- new net PWM3_BO: BIAS_R3.1, OPI_PWM3.COL, P3.3, PWM_R3.1
- new net PWM4_BO: BIAS_R4.1, OPI_PWM4.COL, P4.3, PWM_R4.1
- new net PWM5_BO: BIAS_R5.1, OPI_PWM5.COL, P5.3, PWM_R5.1
- new net PWM6_BO: BIAS_R6.1, OPI_PWM6.COL, P6.3, PWM_R6.1
- new net PWM7_BO: BIAS_R7.1, OPI_PWM7.COL, P7.3, PWM_R7.1
- new net PWM8_BO: BIAS_R8.1, OPI_PWM8.COL, P8.3, PWM_R8.1
- new net PWM9_BO: BIAS_R9.1, OPI_PWM9.COL, P9.3, PWM_R9.1
- net 12V_OUT: now also BIAS_R.2, BIAS_R1.2, BIAS_R2.2, BIAS_R3.2, BIAS_R4.2, BIAS_R5.2, BIAS_R6.2, BIAS_R7.2, BIAS_R8.2, BIAS_R9.2
- net GND: now also OPI_PWM0.C, OPI_PWM1.C, OPI_PWM2.C, OPI_PWM3.C, OPI_PWM4.C, OPI_PWM5.C, OPI_PWM6.C, OPI_PWM7.C, OPI_PWM8.C, OPI_PWM9.C; no longer MICROSD.CD1, MICROSD.CD2
- net GND_ESC: now also OPI_PWM0.EMIT, OPI_PWM1.EMIT, OPI_PWM2.EMIT, OPI_PWM3.EMIT, OPI_PWM4.EMIT, OPI_PWM5.EMIT, OPI_PWM6.EMIT, OPI_PWM7.EMIT, OPI_PWM8.EMIT, OPI_PWM9.EMIT, P0.1, P1.1, P2.1, P3.1, P4.1, P5.1, P6.1, P7.1, P8.1, P9.1; no longer PWM.1, PWM1.1, PWM2.1, PWM3.1, PWM4.1, PWM5.1, PWM6.1, PWM7.1, PWM8.1, PWM9.1
- net PWM0_OUT: now also PWM_IN0.1; no longer PWM.3, PWM_R.1
- net PWM1_OUT: now also PWM_IN1.1; no longer PWM1.3, PWM_R1.1
- net PWM2_OUT: now also PWM_IN2.1; no longer PWM2.3, PWM_R2.1
- net PWM3_OUT: now also PWM_IN3.1; no longer PWM3.3, PWM_R3.1
- net PWM4_OUT: now also PWM_IN4.1; no longer PWM4.3, PWM_R4.1
- net PWM5_OUT: now also PWM_IN5.1; no longer PWM5.3, PWM_R5.1
- net PWM6_OUT: now also PWM_IN6.1; no longer PWM6.3, PWM_R6.1
- net PWM7_OUT: now also PWM_IN7.1; no longer PWM7.3, PWM_R7.1
- net PWM8_OUT: now also PWM_IN8.1; no longer PWM8.3, PWM_R8.1
- net PWM9_OUT: now also PWM_IN9.1; no longer PWM9.3, PWM_R9.1
Other:
- moved on the sheet: PWM_LED, PWM_LED1, PWM_LED2, PWM_LED3, PWM_LED4, PWM_LED5, PWM_LED6, PWM_LED7, PWM_LED8, PWM_LED9, PWM_R, PWM_R1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

Commit message: Small updates before transfer of ownership
Parts:
- removed BIAS_R: 1K, SparkFun-Resistors:0OHM-0603-1/10W-5%
- removed PWM_LED, PWM_LED1, PWM_LED2, PWM_LED3, PWM_LED4, PWM_LED5, PWM_LED6, PWM_LED7, PWM_LED8, PWM_LED9: (no value), SparkFun-LED:LED1206
- removed PWM_R, PWM_R1, PWM_R2, PWM_R3, PWM_R4, PWM_R5, PWM_R6, PWM_R7, PWM_R8, PWM_R9: 330, SparkFun-Resistors:0OHM-0603-1/10W-5%
- added BIAS_R0: 1K, SparkFun-Resistors:0OHM-0603-1/10W-5%
Connections:
- removed net N$13: PWM_LED2.A, PWM_R2.2
- removed net N$14: PWM_LED3.A, PWM_R3.2
- removed net N$18: PWM_LED9.A, PWM_R9.2
- removed net N$19: PWM_LED8.A, PWM_R8.2
- removed net N$20: PWM_LED7.A, PWM_R7.2
- removed net N$21: PWM_LED6.A, PWM_R6.2
- removed net N$22: PWM_LED5.A, PWM_R5.2
- removed net N$26: PWM_LED4.A, PWM_R4.2
- removed net N$7: PWM_LED.A, PWM_R.2
- removed net N$8: PWM_LED1.A, PWM_R1.2
- removed net PWM0_BO: BIAS_R.1, OPI_PWM0.COL, P0.3, PWM_R.1
- removed net PWM1_BO: BIAS_R1.1, OPI_PWM1.COL, P1.3, PWM_R1.1
- removed net PWM2_BO: BIAS_R2.1, OPI_PWM2.COL, P2.3, PWM_R2.1
- removed net PWM3_BO: BIAS_R3.1, OPI_PWM3.COL, P3.3, PWM_R3.1
- removed net PWM4_BO: BIAS_R4.1, OPI_PWM4.COL, P4.3, PWM_R4.1
- removed net PWM5_BO: BIAS_R5.1, OPI_PWM5.COL, P5.3, PWM_R5.1
- removed net PWM6_BO: BIAS_R6.1, OPI_PWM6.COL, P6.3, PWM_R6.1
- removed net PWM7_BO: BIAS_R7.1, OPI_PWM7.COL, P7.3, PWM_R7.1
- removed net PWM8_BO: BIAS_R8.1, OPI_PWM8.COL, P8.3, PWM_R8.1
- removed net PWM9_BO: BIAS_R9.1, OPI_PWM9.COL, P9.3, PWM_R9.1
- new net EMIT0: BIAS_R0.1, OPI_PWM0.EMIT, P0.1
- new net EMIT1: BIAS_R1.1, OPI_PWM1.EMIT, P1.1
- new net EMIT2: BIAS_R2.2, OPI_PWM2.EMIT, P2.1
- new net EMIT3: BIAS_R3.1, OPI_PWM3.EMIT, P3.1
- new net EMIT4: BIAS_R4.1, OPI_PWM4.EMIT, P4.1
- new net EMIT5: BIAS_R5.1, OPI_PWM5.EMIT, P5.1
- new net EMIT6: BIAS_R6.1, OPI_PWM6.EMIT, P6.1
- new net EMIT7: BIAS_R7.1, OPI_PWM7.EMIT, P7.1
- new net EMIT8: BIAS_R8.1, OPI_PWM8.EMIT, P8.1
- new net EMIT9: BIAS_R9.1, OPI_PWM9.EMIT, P9.1
- net 12V_OUT: now also OPI_PWM0.COL, OPI_PWM1.COL, OPI_PWM2.COL, OPI_PWM3.COL, OPI_PWM4.COL, OPI_PWM5.COL, OPI_PWM6.COL, OPI_PWM7.COL, OPI_PWM8.COL, OPI_PWM9.COL, P0.3, P1.3, P2.3, P3.3, P4.3, P5.3, P6.3, P7.3, P8.3, P9.3; no longer BIAS_R.2, BIAS_R1.2, BIAS_R2.2, BIAS_R3.2, BIAS_R4.2, BIAS_R5.2, BIAS_R6.2, BIAS_R7.2, BIAS_R8.2, BIAS_R9.2
- net GND_ESC: now also BIAS_R0.2, BIAS_R1.2, BIAS_R2.1, BIAS_R3.2, BIAS_R4.2, BIAS_R5.2, BIAS_R6.2, BIAS_R7.2, BIAS_R8.2, BIAS_R9.2; no longer OPI_PWM0.EMIT, OPI_PWM1.EMIT, OPI_PWM2.EMIT, OPI_PWM3.EMIT, OPI_PWM4.EMIT, OPI_PWM5.EMIT, OPI_PWM6.EMIT, OPI_PWM7.EMIT, OPI_PWM8.EMIT, OPI_PWM9.EMIT, P0.1, P1.1, P2.1, P3.1, P4.1, P5.1, P6.1, P7.1, P8.1, P9.1, PWM_LED.C, PWM_LED1.C, PWM_LED2.C, PWM_LED3.C, PWM_LED4.C, PWM_LED5.C, PWM_LED6.C, PWM_LED7.C, PWM_LED8.C, PWM_LED9.C
Other:
- moved on the sheet: BIAS_R1, BIAS_R2, BIAS_R3, BIAS_R4, BIAS_R5, BIAS_R6, BIAS_R7, BIAS_R8, BIAS_R9
